File: pcb/gnss_node.kicad_sch (KiCad schematic)
At the start: 0 parts

Commit message: More schematic
Other:
- added sheet IMU (imu.kicad_sch)
Changed lines of the file:
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@@
+	)
+	(sheet
+		(at 217.17 102.87)
+		(size 19.05 15.24)
+		(exclude_from_sim no)
+		(in_bom yes)
+		(on_board yes)
+		(dnp no)
+		(fields_autoplaced yes)
+		(stroke
+			(width 0.1524)
+			(type solid)
+		)
+		(fill
+			(color 0 0 0 0)
+		)
+		(property "Sheetname" "IMU"
+			(at 217.17 102.1584 0)
+			(show_name no)
+			(do_not_autoplace no)
+			(effects
+				(font
+					(size 1.27 1.27)
+				)
+				(justify left bottom)
+			)
+		)
+		(property "Sheetfile" "imu.kicad_sch"
+			(at 217.17 118.6946 0)
+			(show_name no)
+			(do_not_autoplace no)
+			(effects
+				(font
+					(size 1.27 1.27)
+				)
+				(justify left top)
+			)
+		)
+		(instances
+			(project "gnss_node"
+				(path "/eb6e66b6-2df0-4872-8f92-4c510b34f8fe"
+					(page "7")
+				)
+			)
+		)
 	)
 	(sheet

Commit message: routing
Other:
- sheet GPS ports: added GPS_RST; removed none
- sheet IMU ports: added IMU_EN, INT, SCL, SDA; removed none
- sheet MCU ports: added I2C1_SCL, I2C1_SDA, IMU_EN, IMU_INT; removed none
