File: pcb/gnss_node.kicad_pcb (KiCad board)
At the start: 4 copper layers, 86 x 29.9 mm, 112 parts, among them IC1 LT8606IDC#TRPBF, IC2 ATA6561-GAQW-N, IC8 MCP79410T-I_MS, J1 Conn_01x05_Socket, J2 TC2030, J3 Conn_Coaxial_Small, Q1 BSS84, Q2 BSS138, Q3 BSS138, Q4 BC847, U1 STM32L432KCUx, U2 MCP1700x-330xxMB, U3 INA186A4IDCKR, U4 L76L-M33, U701 GAQY212GS, U702 GAQY212GS, Y1 32,768kHz

Commit message: More schematic
Parts:
- moved U4 56.0 mm to (169.6, 38.8), turned to -90 degrees
- moved Q4 43.8 mm to (180.0, 33.9), turned to 180 degrees
- moved R6 24.8 mm to (146.1, 31.7), turned to 180 degrees
- moved J3 23.9 mm to (152.7, 31.5)
- moved D1 23.3 mm to (150.0, 32.5)
- moved C11 6.86 mm to (147.8, 32.1), turned to -90 degrees
- moved C12 5.46 mm to (144.4, 32.1), turned to -90 degrees
- moved Q3 3.03 mm to (140.3, 39.2)
- moved Q1 1.28 mm to (137.9, 34.6)

Commit message: routing
Parts:
- added C54: 220n, Capacitor_SMD:C_0603_1608Metric, B.Cu at (179.0, 81.9)
- added C55: 1u, Capacitor_SMD:C_0603_1608Metric, B.Cu at (183.1, 84.7)
- added C56: 100n, Capacitor_SMD:C_0603_1608Metric, B.Cu at (183.1, 81.7)
- added C57: 100n, Capacitor_SMD:C_0603_1608Metric, B.Cu at (183.1, 83.2)
- added C58: 100n, Capacitor_SMD:C_0603_1608Metric, B.Cu at (153.8, 89.3)
- added C59: 100n, Capacitor_SMD:C_0603_1608Metric, B.Cu at (158.2, 88.4)
- added C60: 1u, Capacitor_SMD:C_0603_1608Metric, B.Cu at (161.3, 88.4)
- added C61: 100n, Capacitor_SMD:C_0603_1608Metric, B.Cu at (150.9, 86.9)
- added C62: 100n, Capacitor_SMD:C_0603_1608Metric, B.Cu at (157.7, 82.7)
- added FB6: 100R @ 100MHz, Inductor_SMD:L_0603_1608Metric, B.Cu at (183.0, 86.9)
- added FB7: 100R @ 100MHz, Inductor_SMD:L_0603_1608Metric, B.Cu at (165.1, 88.8)
- added Q5: BSS138, Package_TO_SOT_SMD:SOT-23, F.Cu at (183.3, 87.2)
- added Q6: BSS84, Package_TO_SOT_SMD:SOT-23, F.Cu at (178.9, 84.9)
- added R33: 10k, Resistor_SMD:R_0603_1608Metric, B.Cu at (175.6, 85.0)
- added R34: 10k, Resistor_SMD:R_0603_1608Metric, B.Cu at (175.6, 83.5)
- added R35: 10k, Resistor_SMD:R_0603_1608Metric, B.Cu at (178.0, 87.6)
- added R36: 10k, Resistor_SMD:R_0603_1608Metric, B.Cu at (179.5, 87.6)
- added R37: 10k, Resistor_SMD:R_0603_1608Metric, B.Cu at (180.5, 84.6)
- added R38: 10k, Resistor_SMD:R_0603_1608Metric, B.Cu at (158.5, 86.3)
- added R39: 10k, Resistor_SMD:R_0603_1608Metric, B.Cu at (158.5, 84.8)
- added R40: 100k, Resistor_SMD:R_0603_1608Metric_Pad0.98x0.95mm_HandSolder, F.Cu at (181.6, 84.9)
- added R41: 100k, Resistor_SMD:R_0603_1608Metric_Pad0.98x0.95mm_HandSolder, F.Cu at (185.9, 87.1)
- added R42: 100k, Resistor_SMD:R_0603_1608Metric_Pad0.98x0.95mm_HandSolder, F.Cu at (184.0, 84.7)
- added U5: FXOS8700CQR1, lib_local:IC_FXOS8700CQR1, B.Cu at (154.2, 86.0)
- added U6: LSM303AGR, lib_local:PQFN50P200X200X100-12N, B.Cu at (178.5, 84.2)
- C11, C12, C45, C46, C47, C49, C50, C51, C52, C53, D1, FB4, FB5, J3, L2, Q1, Q3, R30, R32, R47, R48, R49, R6: moved to B.Cu
- moved R30 65.8 mm to (180.5, 80.2)
- moved R31 64.7 mm to (172.8, 88.3), turned to 90 degrees
- moved Q1 60.4 mm to (180.5, 77.5), turned to 90 degrees
- moved C53 59.7 mm to (182.6, 73.0), turned to 180 degrees
- moved C52 58.8 mm to (181.1, 71.5), turned to 180 degrees
- moved R32 58.4 mm to (180.4, 73.9), turned to 90 degrees
- moved L2 56.1 mm to (182.2, 69.2), turned to 90 degrees
- moved Q3 56.0 mm to (182.8, 75.7), turned to -90 degrees
- moved Q4 54.6 mm to (175.5, 88.3), turned to 0 degrees
- moved R50 53.9 mm to (171.2, 87.7), turned to 90 degrees
- moved R6 49.7 mm to (179.5, 68.4)
- moved J3 49.6 mm to (185.8, 68.4)
- moved C11 49.5 mm to (180.9, 68.9)
- moved C12 49.2 mm to (178.1, 68.0), turned to 90 degrees
- moved D1 48.8 mm to (183.4, 68.2), turned to 90 degrees
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Connections:
- net /MCU/I2C1_SCL renamed /IMU/SCL
- net /MCU/I2C1_SDA renamed /IMU/SDA
- C49 pad 1: Net-(C49-Pad1) -> GND
- C50 pad 2: Net-(C49-Pad1) -> GND
- C51 pad 1: Net-(C49-Pad1) -> GND
- U1 pad 11: /MCU/GPS_RST -> /GPS/GPS_RST
- U1 pad 27: unconnected-(U1-PB4-Pad27) -> /IMU/IMU_EN
- U1 pad 28: unconnected-(U1-PB5-Pad28) -> /IMU/INT
Routing:
- net /GPS/V_BCKP: track 8.40 -> 41.8 mm, vias 0 -> 2
- net /IMU/INT: track 0.00 -> 31.2 mm, vias 0 -> 2
- net /IMU/IMU_EN: track 0.00 -> 29.0 mm, vias 0 -> 2
- net Net-(Q6-D): track 0.00 -> 28.0 mm, vias 0 -> 1
- net /IMU/SCL: track 15.9 -> 43.5 mm
- net Net-(Q4-C): track 0.00 -> 26.9 mm, vias 0 -> 1
- net /GPS/GPS_RX: track 0.76 -> 22.8 mm
- net Net-(U5-SA0/MISO): track 0.00 -> 20.3 mm
- net /GPS/GPS_TX: track 0.00 -> 19.2 mm, vias 0 -> 1
- net /IMU/SDA: track 17.8 -> 36.8 mm
- net /GPS/GPS_PPS: track 2.14 -> 20.3 mm
- net +3.3V: track 78.9 -> 95.4 mm, vias 6 -> 7
- net Net-(Q1-S): track 0.00 -> 11.5 mm
- net Net-(U6-VDD): track 0.00 -> 11.4 mm
- net Net-(U4-V_BCKP): track 0.00 -> 9.35 mm
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Other:
- board size 86 x 29.9 mm -> 76 x 29.9 mm

Commit message: finnishing touches
Parts:
- moved Q4 0.20 mm to (175.5, 88.5)
- moved R31 0.20 mm to (172.8, 88.5)
- moved FB6 0.12 mm to (183.0, 87.0)
Routing:
- net /IMU/SDA: track 36.8 -> 39.8 mm
- net +3.3V: track 95.4 -> 97.6 mm
- net GND: vias 53 -> 54
- net Earth: vias 20 -> 22

Commit message: DRC fixes
Parts:
- moved Q4 1.67 mm to (177.1, 88.0), turned to 90 degrees
Routing:
- net Net-(Q4-B): track 3.77 -> 5.92 mm

Commit message: Unify passive values/footprints, add via-in-pad DRC rule, regen prod outputs
Parts:
- C22, C34: footprint Capacitor_SMD:C_1206_3216Metric_Pad1.33x1.80mm_HandSolder -> Capacitor_SMD:C_1206_3216Metric
- C32, C33, C35, C48: footprint Capacitor_SMD:C_0603_1608Metric_Pad1.08x0.95mm_HandSolder -> Capacitor_SMD:C_0603_1608Metric
- C39: value 4.7nF -> 4.7n; footprint Capacitor_SMD:C_0603_1608Metric_Pad1.08x0.95mm_HandSolder -> Capacitor_SMD:C_0603_1608Metric
- C40, C41: value 4.7pF -> 4.7p; footprint Capacitor_SMD:C_0603_1608Metric_Pad1.08x0.95mm_HandSolder -> Capacitor_SMD:C_0603_1608Metric
- C42, C43: value 6,2p -> 6.2p; footprint Capacitor_SMD:C_0402_1005Metric_Pad0.74x0.62mm_HandSolder -> Capacitor_SMD:C_0402_1005Metric
- R18, R19, R20, R21, R22, R24, R29, R30, R31, R32, R40, R41, R42, R46, R47, R48, R49, R50: footprint Resistor_SMD:R_0603_1608Metric_Pad0.98x0.95mm_HandSolder -> Resistor_SMD:R_0603_1608Metric
- R23: value 560R -> 560; footprint Resistor_SMD:R_0603_1608Metric_Pad0.98x0.95mm_HandSolder -> Resistor_SMD:R_0603_1608Metric
- moved C12 0.15 mm to (177.9, 68.0)
- moved R6 0.07 mm to (179.4, 68.4)
Routing:
- net GND: vias 54 -> 263
