File: pcb/mcu.kicad_sch (KiCad schematic)
At the start: 22 parts, among them IC8 MCP79410T-I_MS, J2 TC2030, U1 STM32L432KCUx, Y1 32,768kHz

Commit message: More schematic
Changed lines of the file:
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@@
+	)
+	(junction
+		(at 115.57 101.6)
+		(diameter 0)
+		(color 0 0 0 0)
 	)
 	(junction
@@
 	(junction
 		(at 132.08 99.06)
+		(diameter 0)
+		(color 0 0 0 0)
+	)
+	(junction
+		(at 115.57 99.06)
 		(diameter 0)
 		(color 0 0 0 0)
@@
 	(wire
 		(pts
+			(xy 114.3 104.14) (xy 115.57 104.14)
+		)
+		(stroke
+			(width 0)
+			(type default)
+		)
+	)
+	(wire
+		(pts
 			(xy 52.07 91.44) (xy 54.61 91.44)
 		)
@@
 	(wire
 		(pts
+			(xy 115.57 101.6) (xy 124.46 101.6)
+		)
+		(stroke
+			(width 0)
+			(type default)
+		)
+	)
+	(wire
+		(pts
 			(xy 52.07 114.3) (xy 57.15 114.3)
 		)
@@
 	(wire
 		(pts
-			(xy 86.36 99.06) (xy 132.08 99.06)
+			(xy 86.36 99.06) (xy 115.57 99.06)
+		)
+		(stroke
+			(width 0)
+			(type default)
+		)
+	)
+	(wire
+		(pts
+			(xy 114.3 95.25) (xy 115.57 95.25)
 		)
 		(stroke
@@
 	(wire
 		(pts
+			(xy 115.57 99.06) (xy 132.08 99.06)
+		)
+		(stroke
+			(width 0)
+			(type default)
+		)
+	)
+	(wire
+		(pts
 			(xy 146.05 58.42) (xy 148.59 58.42)
 		)
@@
 	(wire
 		(pts
-			(xy 86.36 101.6) (xy 124.46 101.6)
+			(xy 86.36 101.6) (xy 115.57 101.6)
 		)
 		(stroke
@@
 	(wire
 		(pts
+			(xy 115.57 104.14) (xy 115.57 101.6)
+		)
+		(stroke
+			(width 0)
+			(type default)
+		)
+	)
+	(wire
+		(pts
 			(xy 148.59 114.3) (xy 148.59 115.57)
 		)
@@
 		(pts
 			(xy 57.15 114.3) (xy 60.96 114.3)
+		)
+		(stroke
+			(width 0)
+			(type default)
+		)
+	)
+	(wire
+		(pts
+			(xy 115.57 95.25) (xy 115.57 99.06)
 		)
 		(stroke
@@
 		)
 	)
-	(label "I2C1_SDA"
-		(at 114.3 101.6 0)
-		(effects
-			(font
-				(size 1.27 1.27)
-			)
-			(justify left bottom)
-		)
-	)
 	(label "SWCLK"
 		(at 165.1 104.14 0)
@@
 		)
 	)
-	(label "I2C1_SCL"
-		(at 114.3 99.06 0)
-		(effects
-			(font
-				(size 1.27 1.27)
-			)
-			(justify left bottom)
-		)
-	)
 	(label "Y1-"
 		(at 54.61 99.06 0)
@@
 			)
 			(justify left bottom)
+		)
+	)
+	(hierarchical_label "I2C1_SDA"
+		(shape input)
+		(at 114.3 104.14 180)
+		(effects
+			(font
+				(size 1.27 1.27)
+			)
+			(justify right)
 		)
 	)
@@
 		)
 	)
+	(hierarchical_label "I2C1_SCL"
+		(shape input)
+		(at 114.3 95.25 180)
+		(effects
+			(font
+				(size 1.27 1.27)
+			)
+			(justify right)
+		)
+	)

Commit message: routing
Connections:
- net IMU_EN: now reaches U1.27 (PB4)
- net IMU_INT: now reaches U1.28 (PB5)
- no-connect marks 7 -> 5
Changed lines of the file:
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@@
-	)
-	(no_connect
-		(at 135.89 96.52)
 	)
 	(no_connect
@@
 	)
 	(no_connect
-		(at 135.89 93.98)
-	)
-	(no_connect
 		(at 161.29 68.58)
 	)
@@
 	(wire
 		(pts
+			(xy 129.54 93.98) (xy 135.89 93.98)
+		)
+		(stroke
+			(width 0)
+			(type default)
+		)
+	)
+	(wire
+		(pts
 			(xy 132.08 113.03) (xy 132.08 114.3)
 		)
@@
 		(pts
 			(xy 78.74 114.3) (xy 82.55 114.3)
+		)
+		(stroke
+			(width 0)
+			(type default)
+		)
+	)
+	(wire
+		(pts
+			(xy 129.54 96.52) (xy 135.89 96.52)
 		)
 		(stroke
@@
 		)
 	)
+	(hierarchical_label "IMU_INT"
+		(shape input)
+		(at 129.54 96.52 180)
+		(effects
+			(font
+				(size 1.27 1.27)
+			)
+			(justify right)
+		)
+	)
 	(hierarchical_label "V_BCKP"
 		(shape input)
@@
 		)
 	)
+	(hierarchical_label "IMU_EN"
+		(shape output)
+		(at 129.54 93.98 180)
+		(effects
+			(font
+				(size 1.27 1.27)
+			)
+			(justify right)
+		)
+	)

Commit message: Unify passive values/footprints, add via-in-pad DRC rule, regen prod outputs
Parts:
- C42, C43: value 6,2p -> 6.2p; footprint Capacitor_SMD:C_0402_1005Metric_Pad0.74x0.62mm_HandSolder -> Capacitor_SMD:C_0402_1005Metric
- C48: footprint Capacitor_SMD:C_0603_1608Metric_Pad1.08x0.95mm_HandSolder -> Capacitor_SMD:C_0603_1608Metric
- R18, R19, R20, R29, R46: footprint Resistor_SMD:R_0603_1608Metric_Pad0.98x0.95mm_HandSolder -> Resistor_SMD:R_0603_1608Metric
Changed lines of the file:
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@@
 			)
 		)
-		(property "Footprint" "Resistor_SMD:R_0603_1608Metric_Pad0.98x0.95mm_HandSolder"
+		(property "Footprint" "Resistor_SMD:R_0603_1608Metric"
 			(at 167.64 104.902 90)
 			(hide yes)
@@
 			)
 		)
-		(property "Footprint" "Resistor_SMD:R_0603_1608Metric_Pad0.98x0.95mm_HandSolder"
+		(property "Footprint" "Resistor_SMD:R_0603_1608Metric"
 			(at 64.77 116.078 90)
 			(hide yes)
@@
 			)
 		)
-		(property "Footprint" "Resistor_SMD:R_0603_1608Metric_Pad0.98x0.95mm_HandSolder"
+		(property "Footprint" "Resistor_SMD:R_0603_1608Metric"
 			(at 130.302 109.22 90)
 			(hide yes)
@@
 			)
 		)
-		(property "Footprint" "Resistor_SMD:R_0603_1608Metric_Pad0.98x0.95mm_HandSolder"
+		(property "Footprint" "Resistor_SMD:R_0603_1608Metric"
 			(at 122.682 109.22 90)
 			(hide yes)
@@
 			)
 		)
-		(property "Footprint" "Resistor_SMD:R_0603_1608Metric_Pad0.98x0.95mm_HandSolder"
+		(property "Footprint" "Resistor_SMD:R_0603_1608Metric"
 			(at 85.852 88.9 90)
 			(hide yes)
@@
 			)
 		)
-		(property "Footprint" "Capacitor_SMD:C_0603_1608Metric_Pad1.08x0.95mm_HandSolder"
+		(property "Footprint" "Capacitor_SMD:C_0603_1608Metric"
 			(at 91.1352 111.76 0)
 			(hide yes)
@@
 			)
 		)
-		(property "Value" "6,2p"
+		(property "Value" "6.2p"
 			(at 41.402 92.964 90)
 			(show_name no)
@@
 			)
 		)
-		(property "Footprint" "Capacitor_SMD:C_0402_1005Metric_Pad0.74x0.62mm_HandSolder"
+		(property "Footprint" "Capacitor_SMD:C_0402_1005Metric"
 			(at 49.53 90.4748 0)
 			(hide yes)
@@
 			)
 		)
-		(property "Value" "6,2p"
+		(property "Value" "6.2p"
 			(at 41.91 100.584 90)
 			(show_name no)
@@
 			)
 		)
-		(property "Footprint" "Capacitor_SMD:C_0402_1005Metric_Pad0.74x0.62mm_HandSolder"
+		(property "Footprint" "Capacitor_SMD:C_0402_1005Metric"
 			(at 49.53 98.0948 0)
 			(hide yes)
