File: pcb/prot.kicad_sch (KiCad schematic)
At the start: 17 parts, among them J1 Conn_01x05_Socket

Commit message: Unify passive values/footprints, add via-in-pad DRC rule, regen prod outputs
Parts:
- C22: footprint Capacitor_SMD:C_1206_3216Metric_Pad1.33x1.80mm_HandSolder -> Capacitor_SMD:C_1206_3216Metric
Changed lines of the file:
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@@
 			)
 		)
-		(property "Footprint" "Capacitor_SMD:C_1206_3216Metric_Pad1.33x1.80mm_HandSolder"
+		(property "Footprint" "Capacitor_SMD:C_1206_3216Metric"
 			(at 67.31 134.3152 0)
 			(hide yes)
